Commit message: edit starting joint positings for pick and place, while still keeping on pi range

File: urdf/inc/ur_joint_control.xacro (robot description, xacro)
@@ -8,4 +8,5 @@
       <command_interface name="position"/>
       <command_interface name="velocity"/>
+      <command_interface name="effort"/>
       <state_interface name="position">
         <!-- initial position for the mock system and simulation -->
@@ -22,4 +23,5 @@
       <command_interface name="position"/>
       <command_interface name="velocity"/>
+      <command_interface name="effort"/>
       <state_interface name="position">
         <!-- initial position for the mock system and simulation -->
@@ -36,4 +38,5 @@
       <command_interface name="position"/>
       <command_interface name="velocity"/>
+      <command_interface name="effort"/>
       <state_interface name="position">
         <!-- initial position for the mock system and simulation -->
@@ -50,4 +53,5 @@
       <command_interface name="position"/>
       <command_interface name="velocity"/>
+      <command_interface name="effort"/>
       <state_interface name="position">
         <!-- initial position for the mock system and simulation -->
@@ -64,4 +68,5 @@
       <command_interface name="position"/>
       <command_interface name="velocity"/>
+      <command_interface name="effort"/>
       <state_interface name="position">
         <!-- initial position for the mock system and simulation -->
@@ -78,4 +83,5 @@
       <command_interface name="position"/>
       <command_interface name="velocity"/>
+      <command_interface name="effort"/>
       <state_interface name="position">
         <!-- initial position for the mock system and simulation -->

File: urdf/ur_macro.xacro (robot description, xacro)
@@ -306,5 +306,5 @@
          <safety_controller soft_lower_limit="${shoulder_pan_lower_limit + safety_pos_margin}" soft_upper_limit="${shoulder_pan_upper_limit - safety_pos_margin}" k_position="${safety_k_position}" k_velocity="0.0"/>
       </xacro:if>
-      <dynamics damping="0" friction="0"/>
+      <dynamics damping="0.2" friction="0.5"/>
     </joint>
     <joint name="${tf_prefix}shoulder_lift_joint" type="revolute">
@@ -318,5 +318,5 @@
          <safety_controller soft_lower_limit="${shoulder_lift_lower_limit + safety_pos_margin}" soft_upper_limit="${shoulder_lift_upper_limit - safety_pos_margin}" k_position="${safety_k_position}" k_velocity="0.0"/>
       </xacro:if>
-      <dynamics damping="0" friction="0"/>
+      <dynamics damping="0.2" friction="0.5"/>
     </joint>
     <joint name="${tf_prefix}elbow_joint" type="revolute">
@@ -330,5 +330,5 @@
          <safety_controller soft_lower_limit="${elbow_joint_lower_limit + safety_pos_margin}" soft_upper_limit="${elbow_joint_upper_limit - safety_pos_margin}" k_position="${safety_k_position}" k_velocity="0.0"/>
       </xacro:if>
-      <dynamics damping="0" friction="0"/>
+      <dynamics damping="0.2" friction="0.5"/>
     </joint>
     <joint name="${tf_prefix}wrist_1_joint" type="revolute">
@@ -342,5 +342,5 @@
          <safety_controller soft_lower_limit="${wrist_1_lower_limit + safety_pos_margin}" soft_upper_limit="${wrist_1_upper_limit - safety_pos_margin}" k_position="${safety_k_position}" k_velocity="0.0"/>
       </xacro:if>
-      <dynamics damping="0" friction="0"/>
+      <dynamics damping="0.2" friction="0.5"/>
     </joint>
     <joint name="${tf_prefix}wrist_2_joint" type="revolute">
@@ -354,5 +354,5 @@
          <safety_controller soft_lower_limit="${wrist_2_lower_limit + safety_pos_margin}" soft_upper_limit="${wrist_2_upper_limit - safety_pos_margin}" k_position="${safety_k_position}" k_velocity="0.0"/>
       </xacro:if>
-      <dynamics damping="0" friction="0"/>
+      <dynamics damping="0.2" friction="0.5"/>
     </joint>
     <joint name="${tf_prefix}wrist_3_joint" type="${wrist_3_joint_type}">
@@ -374,5 +374,5 @@
         </xacro:if>
       </xacro:unless>
-      <dynamics damping="0" friction="0"/>
+      <dynamics damping="0.2" friction="0.5"/>
     </joint>
     <link name="${tf_prefix}ft_frame"/>
