Commit message: ss

File: urdf/inc/ur_common.xacro (robot description, xacro)
@@ -11,5 +11,5 @@
     Contributor: Felix Messmer
   -->
-  <xacro:macro name="cylinder_inertial" params="radius length mass *origin">
+  <xacro:macro name="cylinder_inertial_ur" params="radius length mass *origin">
     <inertial>
       <mass value="${mass}" />

File: urdf/ur_config.urdf.xacro (robot description, xacro)
@@ -2,17 +2,19 @@
 <robot xmlns:xacro="http://wiki.ros.org/xacro" name="ur">
    <xacro:include filename="$(find ur_description)/urdf/ur_macro.xacro"/>
-   <xacro:arg name="config_file" default="$(find ur_description)/urdf/config/ex_make_arm.yaml"/>
-   <xacro:property name="config_file" value="$(arg config_file)"/>
-   <xacro:property name="cfg" value="${xacro.load_yaml(config_file)}"/>
+   <xacro:arg name="config_file_path" default="$(find ur_description)/urdf/config/ex_make_arm.yaml"/>
+   <xacro:property name="config_file_path" value="$(arg config_file_path)"/>
+   <xacro:property name="cfg" value="${xacro.load_yaml(config_file_path)}"/>
    <link name="world"/>
-   <joint name="world_to_base_link" type="fixed">
-    <parent link="world"/>
-    <child link="base_link"/>
-  </joint>
-   <link name="base_link"/>
-   <joint name="base_link_to_base_link_ur" type="fixed">
-      <parent link="base_link"/>
-      <child link="base_link_ur"/>
-    </joint>
-   <xacro:make_arm config_file="${config_file}"/>
+   <joint name="world_to_base" type="fixed">
+       <origin xyz="${cfg['world_xyz']}" rpy="${cfg['world_rpy']}"/>
+       <parent link="world"/>
+       <child link="base_link"/>
+   </joint>
+  <link name="base_link"/>
+   <joint name="base_link_joint" type="fixed">
+       <origin xyz="${cfg['base_xyz']}" rpy="${cfg['base_rpy']}"/>
+       <parent link="base_link"/>
+       <child link="${cfg['prefix']}base_link_ur"/>
+   </joint>
+   <xacro:make_arm config_file_path="${config_file_path}"/>
 </robot>

File: urdf/ur_macro.xacro (robot description, xacro)
@@ -89,7 +89,7 @@
         </geometry>
       </collision>
-      <xacro:cylinder_inertial radius="${base_inertia_radius}" length="${base_inertia_length}" mass="${base_mass}">
+      <xacro:cylinder_inertial_ur radius="${base_inertia_radius}" length="${base_inertia_length}" mass="${base_mass}">
         <origin xyz="0 0 0" rpy="0 0 0" />
-      </xacro:cylinder_inertial>
+      </xacro:cylinder_inertial_ur>
     </link>
     <link name="${tf_prefix}shoulder_link">
@@ -376,4 +376,5 @@
       <dynamics damping="0.05" friction="0.1"/>
     </joint>
+      <!-- The FT Frame has the same pose as tool0_flip, but we add tool0_flip because its more verbose -->
     <link name="${tf_prefix}ft_frame"/>
     <joint name="${tf_prefix}wrist_3_link-ft_frame" type="fixed">
@@ -425,12 +426,18 @@
       <origin xyz="0 0 0.1" rpy="${pi} 0 0" />
     </joint>
+      <link name="${tf_prefix}tool0_flip"/>
+      <joint name="${tf_prefix}tool0-tool0flip" type="fixed">
+        <origin xyz="0 0 0" rpy="${pi} 0 0"/>
+        <parent link="${tf_prefix}tool0"/>
+        <child link="${tf_prefix}tool0_flip"/>
+      </joint>
   </xacro:macro>
-  <xacro:macro name="make_arm" params="config_file">
-    <xacro:property name="cfg" value="${xacro.load_yaml(config_file)}"/>
+  <xacro:macro name="make_arm" params="config_file_path">
+    <xacro:property name="cfg" value="${xacro.load_yaml(config_file_path)}"/>
     <xacro:arg name="name" default="ur"/>
-    <xacro:arg name="ur_type" default="${cfg['urdf']['xacro_args']['ur_type']}"/>
+    <xacro:arg name="ur_type" default="${cfg['info']['sku']}"/>
     <!-- parameters -->
     <!-- <xacro:arg name="tf_prefix" default="${cfg['urdf']['xacro_args']['tf_prefix']}" /> -->
-    <xacro:arg name="tf_prefix" default="''" />
+    <xacro:arg name="tf_prefix" default="${cfg['prefix']}" />
     <xacro:arg name="joint_limit_params" default="$(find ur_description)/config/$(arg ur_type)/joint_limits.yaml"/>
     <xacro:arg name="kinematics_params" default="$(find ur_description)/config/$(arg ur_type)/default_kinematics.yaml"/>
