Commit message: refactored so that it can be used with config file and add base_link_ur

File: urdf/ur.urdf.xacro (robot description, xacro)
@@ -1,4 +1,4 @@
 <?xml version="1.0"?>
-<robot xmlns:xacro="http://wiki.ros.org/xacro" name="$(arg name)">
+<robot xmlns:xacro="http://wiki.ros.org/xacro" name="ur">
    <!-- robot name parameter -->
    <xacro:arg name="name" default="ur"/>
@@ -7,5 +7,6 @@
    <!-- possible 'ur_type' values: ur3, ur3e, ur5, ur5e, ur7e, ur10, ur10e, ur12e, ur16e, ur15, ur20, ur30 -->
    <!-- the default value should raise an error in case this was called without defining the type -->
-   <xacro:arg name="ur_type" default="ur5x"/>
+   <!-- <xacro:arg name="ur_type" default="ur5x"/> -->
+   <xacro:arg name="ur_type" default="ur5e"/>
    <!-- parameters -->
    <xacro:arg name="tf_prefix" default="" />
@@ -21,10 +22,18 @@
    <xacro:arg name="force_abs_paths" default="false" />
    <!-- create link fixed to the "world" -->
-   <link name="world" />
+   <link name="world"/>
+   <joint name="world_to_base_link" type="fixed">
+    <parent link="world"/>
+    <child link="base_link"/>
+  </joint>
+   <link name="base_link"/>
+   <joint name="base_link_to_base_link_ur" type="fixed">
+    <parent link="base_link"/>
+    <child link="base_link_ur"/>
+  </joint>
    <!-- arm -->
    <xacro:ur_robot
      name="$(arg name)"
      tf_prefix="$(arg tf_prefix)"
-     parent="world"
      joint_limits_parameters_file="$(arg joint_limit_params)"
      kinematics_parameters_file="$(arg kinematics_params)"
@@ -35,6 +44,4 @@
      safety_k_position="$(arg safety_k_position)"
      force_abs_paths="$(arg force_abs_paths)"
-     >
-     <origin xyz="0 0 0" rpy="0 0 0" />          <!-- position robot in the world -->
-   </xacro:ur_robot>
+     />
 </robot>

File: urdf/ur_macro.xacro (robot description, xacro)
@@ -46,6 +46,4 @@
     name
     tf_prefix
-    parent
-    *origin
     joint_limits_parameters_file
     kinematics_parameters_file
@@ -65,5 +63,5 @@
       force_abs_paths="${force_abs_paths}"/>
     <!-- links -  main serial chain -->
-    <!-- base_link serves as the root of the robot's kinematic tree. It follows REP-103
+    <!-- base_link_ur serves as the root of the robot's kinematic tree. It follows REP-103
         conventions (i.e., X+ forward, Y+ left, Z+ up).
         Since some kinematic solvers forbid having inertia values attached to a root link, we've
@@ -71,5 +69,6 @@
         information.
     -->
-    <link name="${tf_prefix}base_link"/>
+    <!-- Rename base_link to base_link_ur so you can add another base_link_ur outside... -->
+    <link name="${tf_prefix}base_link_ur"/>
     <link name="${tf_prefix}base_link_inertia">
       <xacro:get_visual_params name="base" type="mesh_offset"/>
@@ -279,17 +278,17 @@
       </inertial>
     </link>
-    <!-- base_joint fixes base_link to the environment -->
-    <joint name="${tf_prefix}base_joint" type="fixed">
+    <!-- base_joint fixes base_link_ur to the environment -->
+    <!-- <joint name="${tf_prefix}base_joint" type="fixed">
       <xacro:insert_block name="origin" />
       <parent link="${parent}" />
-      <child link="${tf_prefix}base_link" />
-    </joint>
+      <child link="${tf_prefix}base_link_ur" />
+    </joint> -->
     <!-- joints - main serial chain -->
-    <joint name="${tf_prefix}base_link-base_link_inertia" type="fixed">
-      <parent link="${tf_prefix}base_link" />
+    <joint name="${tf_prefix}base_link_ur-base_link_inertia" type="fixed">
+      <parent link="${tf_prefix}base_link_ur" />
       <child link="${tf_prefix}base_link_inertia" />
-      <!-- 'base_link' is REP-103 aligned (so X+ forward), while the internal
+      <!-- 'base_link_ur' is REP-103 aligned (so X+ forward), while the internal
            frames of the robot/controller have X+ pointing backwards.
-           Use the joint between 'base_link' and 'base_link_inertia' (a dummy
+           Use the joint between 'base_link_ur' and 'base_link_inertia' (a dummy
            link/frame) to introduce the necessary rotation over Z (of pi rad).
       -->
@@ -306,5 +305,6 @@
          <safety_controller soft_lower_limit="${shoulder_pan_lower_limit + safety_pos_margin}" soft_upper_limit="${shoulder_pan_upper_limit - safety_pos_margin}" k_position="${safety_k_position}" k_velocity="0.0"/>
       </xacro:if>
-      <dynamics damping="0.2" friction="0.5"/>
+      <!-- Increase friction in lower joints, they seem to be osscilating alot in sim, and we know friction increases with load -->
+      <dynamics damping="0.05" friction="0.3"/>
     </joint>
     <joint name="${tf_prefix}shoulder_lift_joint" type="revolute">
@@ -318,5 +318,5 @@
          <safety_controller soft_lower_limit="${shoulder_lift_lower_limit + safety_pos_margin}" soft_upper_limit="${shoulder_lift_upper_limit - safety_pos_margin}" k_position="${safety_k_position}" k_velocity="0.0"/>
       </xacro:if>
-      <dynamics damping="0.2" friction="0.5"/>
+      <dynamics damping="0.05" friction="0.3"/>
     </joint>
     <joint name="${tf_prefix}elbow_joint" type="revolute">
@@ -330,5 +330,5 @@
          <safety_controller soft_lower_limit="${elbow_joint_lower_limit + safety_pos_margin}" soft_upper_limit="${elbow_joint_upper_limit - safety_pos_margin}" k_position="${safety_k_position}" k_velocity="0.0"/>
       </xacro:if>
-      <dynamics damping="0.2" friction="0.5"/>
+      <dynamics damping="0.05" friction="0.1"/>
     </joint>
     <joint name="${tf_prefix}wrist_1_joint" type="revolute">
@@ -342,5 +342,5 @@
          <safety_controller soft_lower_limit="${wrist_1_lower_limit + safety_pos_margin}" soft_upper_limit="${wrist_1_upper_limit - safety_pos_margin}" k_position="${safety_k_position}" k_velocity="0.0"/>
       </xacro:if>
-      <dynamics damping="0.2" friction="0.5"/>
+      <dynamics damping="0.05" friction="0.1"/>
     </joint>
     <joint name="${tf_prefix}wrist_2_joint" type="revolute">
@@ -354,5 +354,5 @@
          <safety_controller soft_lower_limit="${wrist_2_lower_limit + safety_pos_margin}" soft_upper_limit="${wrist_2_upper_limit - safety_pos_margin}" k_position="${safety_k_position}" k_velocity="0.0"/>
       </xacro:if>
-      <dynamics damping="0.2" friction="0.5"/>
+      <dynamics damping="0.05" friction="0.1"/>
     </joint>
     <joint name="${tf_prefix}wrist_3_joint" type="${wrist_3_joint_type}">
@@ -374,5 +374,5 @@
         </xacro:if>
       </xacro:unless>
-      <dynamics damping="0.2" friction="0.5"/>
+      <dynamics damping="0.05" friction="0.1"/>
     </joint>
     <link name="${tf_prefix}ft_frame"/>
@@ -382,8 +382,8 @@
       <origin xyz="0 0 0" rpy="${pi} 0 0"/>
     </joint>
-    <!-- ROS-Industrial 'base' frame - base_link to UR 'Base' Coordinates transform -->
+    <!-- ROS-Industrial 'base' frame - base_link_ur to UR 'Base' Coordinates transform -->
     <link name="${tf_prefix}base"/>
-    <joint name="${tf_prefix}base_link-base_fixed_joint" type="fixed">
-      <!-- Note the rotation over Z of pi radians - as base_link is REP-103
+    <joint name="${tf_prefix}base_link_ur-base_fixed_joint" type="fixed">
+      <!-- Note the rotation over Z of pi radians - as base_link_ur is REP-103
            aligned (i.e., has X+ forward, Y+ left and Z+ up), this is needed
            to correctly align 'base' with the 'Base' coordinate system of
@@ -391,5 +391,5 @@
       -->
       <origin xyz="0 0 0" rpy="0 0 ${pi}"/>
-      <parent link="${tf_prefix}base_link"/>
+      <parent link="${tf_prefix}base_link_ur"/>
       <child link="${tf_prefix}base"/>
     </joint>
@@ -417,4 +417,42 @@
       <origin xyz="0 0 0" rpy="0.0 ${-pi/2.0} ${pi/2.0}" />
     </joint>
+    <!-- For testing IK offset converions, helpful to have a offset tcp link -->
+    <link name="${tf_prefix}tcp_world_test" />
+    <joint name="${tf_prefix}tool0_to_tcp_world_test" type="fixed">
+      <parent link="${tf_prefix}tool0" />
+      <child link="${tf_prefix}tcp_world_test" />
+      <!-- Go forward a bit along z and flip around -->
+      <origin xyz="0 0 0.1" rpy="${pi} 0 0" />
+    </joint>
+  </xacro:macro>
+  <xacro:macro name="make_arm" params="config_file">
+    <xacro:property name="cfg" value="${xacro.load_yaml(config_file)}"/>
+    <xacro:arg name="name" default="ur"/>
+    <xacro:arg name="ur_type" default="${cfg['urdf']['xacro_args']['ur_type']}"/>
+    <!-- parameters -->
+    <!-- <xacro:arg name="tf_prefix" default="${cfg['urdf']['xacro_args']['tf_prefix']}" /> -->
+    <xacro:arg name="tf_prefix" default="''" />
+    <xacro:arg name="joint_limit_params" default="$(find ur_description)/config/$(arg ur_type)/joint_limits.yaml"/>
+    <xacro:arg name="kinematics_params" default="$(find ur_description)/config/$(arg ur_type)/default_kinematics.yaml"/>
+    <xacro:arg name="physical_params" default="$(find ur_description)/config/$(arg ur_type)/physical_parameters.yaml"/>
+    <xacro:arg name="visual_params" default="$(find ur_description)/config/$(arg ur_type)/visual_parameters.yaml"/>
+    <xacro:arg name="transmission_hw_interface" default=""/>
+    <xacro:arg name="safety_limits" default="false"/>
+    <xacro:arg name="safety_pos_margin" default="0.15"/>
+    <xacro:arg name="safety_k_position" default="20"/>
+    <!--When using gazebo simulations absolute paths are necessary.-->
+    <xacro:arg name="force_abs_paths" default="false" />
+    <xacro:ur_robot
+      name="$(arg name)"
+      tf_prefix="$(arg tf_prefix)"
+      joint_limits_parameters_file="$(arg joint_limit_params)"
+      kinematics_parameters_file="$(arg kinematics_params)"
+      physical_parameters_file="$(arg physical_params)"
+      visual_parameters_file="$(arg visual_params)"
+      safety_limits="$(arg safety_limits)"
+      safety_pos_margin="$(arg safety_pos_margin)"
+      safety_k_position="$(arg safety_k_position)"
+      force_abs_paths="$(arg force_abs_paths)"
+      />
   </xacro:macro>
 </robot>
