Commit message: ss

File: urdf/ur_config.urdf.xacro (robot description, xacro)
@@ -3,10 +3,10 @@
    <xacro:arg name="ur_description" default="$(env UR_DESCRIPTION_PATH)"/>
    <xacro:include filename="$(arg ur_description)/urdf/ur_macro.xacro"/>
-   <xacro:arg name="config_file_path" default="$(arg ur_description)/urdf/config/ex_make_arm.yaml"/>
-   <xacro:property name="config_file_path" value="$(arg config_file_path)"/>
-   <xacro:property name="cfg" value="${xacro.load_yaml(config_file_path)}"/>
+   <xacro:arg name="config_file" default="$(arg ur_description)/urdf/config/ex_make_arm.yaml"/>
+   <xacro:property name="config_file" value="$(arg config_file)"/>
+   <xacro:property name="cfg" value="${xacro.load_yaml(config_file)}"/>
    <link name="world"/>
    <joint name="world_to_base" type="fixed">
-       <origin xyz="${cfg['world_xyz']}" rpy="${cfg['world_rpy']}"/>
+       <origin xyz="${cfg['args']['world_xyz']}" rpy="${cfg['args']['world_rpy']}"/>
        <parent link="world"/>
        <child link="base_link"/>
@@ -14,8 +14,8 @@
   <link name="base_link"/>
    <joint name="base_link_joint" type="fixed">
-       <origin xyz="${cfg['base_xyz']}" rpy="${cfg['base_rpy']}"/>
+       <origin xyz="${cfg['args']['base_xyz']}" rpy="${cfg['args']['base_rpy']}"/>
        <parent link="base_link"/>
-       <child link="${cfg['prefix']}base_link_ur"/>
+       <child link="${cfg['info']['prefix']}base_link_ur"/>
    </joint>
-   <xacro:make_arm config_file_path="${config_file_path}"/>
+   <xacro:make_arm config_file="${config_file}"/>
 </robot>

File: urdf/ur_macro.xacro (robot description, xacro)
@@ -434,11 +434,11 @@
       </joint>
   </xacro:macro>
-  <xacro:macro name="make_arm" params="config_file_path">
-    <xacro:property name="cfg" value="${xacro.load_yaml(config_file_path)}"/>
+  <xacro:macro name="make_arm" params="config_file">
+    <xacro:property name="cfg" value="${xacro.load_yaml(config_file)}"/>
     <xacro:arg name="name" default="ur"/>
     <xacro:arg name="ur_type" default="${cfg['info']['sku']}"/>
     <!-- parameters -->
     <!-- <xacro:arg name="tf_prefix" default="${cfg['urdf']['xacro_args']['tf_prefix']}" /> -->
-    <xacro:arg name="tf_prefix" default="${cfg['prefix']}" />
+    <xacro:arg name="tf_prefix" default="${cfg['info']['prefix']}" />
     <xacro:arg name="joint_limit_params" default="$(arg ur_description)/config/$(arg ur_type)/joint_limits.yaml"/>
     <xacro:arg name="kinematics_params" default="$(arg ur_description)/config/$(arg ur_type)/default_kinematics.yaml"/>
