Commit message: added support for closed form kinematics

File: urdf/ur_macro.xacro (robot description, xacro)
@@ -409,4 +409,12 @@
       <child link="${tf_prefix}tool0"/>
     </joint>
+    <!-- https://github.com/ros-industrial/universal_robot/pull/506/files -->
+    <!-- Link from original ur_kinematics, see notes in the ur_ros1 package-->
+    <link name="${tf_prefix}ee_link"/>
+    <joint name="${tf_prefix}ee_fixed_joint" type="fixed">
+      <parent link="${tf_prefix}wrist_3_link" />
+      <child link="${tf_prefix}ee_link" />
+      <origin xyz="0 0 0" rpy="0.0 ${-pi/2.0} ${pi/2.0}" />
+    </joint>
   </xacro:macro>
 </robot>

Commit message: ss

File: urdf/ur_macro.xacro (robot description, xacro)
@@ -434,4 +434,7 @@
       </joint>
   </xacro:macro>
+  <xacro:macro name="make_config" params="config_file">
+    <xacro:make_arm config_file="${config_file}"/>
+  </xacro:macro>
   <xacro:macro name="make_arm" params="config_file">
     <xacro:property name="cfg" value="${xacro.load_yaml(config_file)}"/>
